File: Teebeutel.sch (KiCad schematic (older format))
At the start: 163 parts, among them J1 RJ45_Shielded, J2 Battery, J3 Micro_SD_Card, J4 Conn_01x30_Female, J5 Conn_01x10_Female, J6 Conn_01x10_Female, M1 Motor_DC, Q1 S8050, Q2 S8050, Q3 AO3400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

Commit message: feat(): Change footprints
Parts:
- removed U11: TLV1117-33, Package_TO_SOT_SMD:SOT-223, symbol Regulator_Linear:TLV1117-33
- added L2: 2.2µH, Inductor_SMD:L_1210_3225Metric, symbol Device:L
- added R36: 900kΩ, Resistor_SMD:R_0603_1608Metric, symbol Device:R
- added R37: 200KΩ, Resistor_SMD:R_0603_1608Metric, symbol Device:R
- added U11: TLV62568DBV, Package_TO_SOT_SMD:SOT-23-5, symbol Regulator_Switching:TLV62568DBV
- U13: footprint Teebeutel_Special_Parts:QFN50P400X400X100-25N-D -> Package_SO:TSSOP-24_4.4x7.8mm_P0.65mm; symbol Teebeutel_Special_Parts:PCA9539BS,118 -> Teebeutel_Special_Parts:PCA9539D_PW; LCSC C2669675 -> C129516
- U4, U9: footprint Package_DFN_QFN:Texas_R_PUQFN-N12 -> Package_SO:TSSOP-14_4.4x5mm_P0.65mm; symbol Logic_LevelTranslator:TXB0104RUT -> Logic_LevelTranslator:TXB0104PW; JLC UQFN-12_1.7x2.0x0.4P -> (none); LCSC C105266 -> C60708
Connections:
- net +1V8: now also U9.14 (VCCB); no longer U9.11 (VCCB)
- net +3V3: now also U13.24 (VDD), U4.14 (VCCB), L2.2, R36.1; no longer U13.21 (VDD), U4.11 (VCCB)
- net +BATT: now also U11.1 (EN), U11.4 (VIN)
- net BTN_DOWN: now also U13.6 (IO0_2); no longer U13.3 (IO0_2)
- net BTN_LEFT: now also U13.7 (IO0_3); no longer U13.4 (IO0_3)
- net BTN_PUSH: now also U13.4 (IO0_0); no longer U13.1 (IO0_0)
- net BTN_RIGHT: now also U13.8 (IO0_4); no longer U13.5 (IO0_4)
- net BTN_UP: now also U13.5 (IO0_1); no longer U13.2 (IO0_1)
- net DTR: now also U4.13 (B1); no longer U4.10 (B1)
- net EXP-IO0-8: now also U13.11 (IO0_7); no longer U13.8 (IO0_7)
- net EXP-IO1-0: now also U13.13 (IO1_0); no longer U13.10 (IO1_0)
- net EXP-IO1-1: now also U13.14 (IO1_1); no longer U13.11 (IO1_1)
- net EXP-IO1-2: now also U13.15 (IO1_2); no longer U13.12 (IO1_2)
- net EXP-IO1-3: now also U13.16 (IO1_3); no longer U13.13 (IO1_3)
- net EXP-IO1-4: now also U13.17 (IO1_4); no longer U13.14 (IO1_4)
- net EXP-IO1-5: now also U13.18 (IO1_5); no longer U13.15 (IO1_5)
- net EXP-IO1-6: now also U13.19 (IO1_6); no longer U13.16 (IO1_6)
- net EXP-IO1-7: now also U13.20 (IO1_7); no longer U13.17 (IO1_7)
- net EXP-~INT: now also U13.1 (~INT); no longer U13.22 (~INT)
- net EXP-~RST: now also U13.3 (~RESET); no longer U13.24 (~RESET)
- net GND: now also U13.12 (VSS), U4.7 (GND), U9.7 (GND), R37.2, U11.2 (GND); no longer U13.25 (EP), U13.9 (VSS), U4.6 (GND), U9.6 (GND)
- net I2C-SCL: now also U13.22 (SDA); no longer U13.19 (SCL)
- net I2C-SDA: now also U13.22 (SDA); no longer U13.20 (SDA)
- net RTS: now also U4.10 (B4); no longer U4.7 (B4)
- net RxD: now also U4.11 (B3); no longer U4.8 (B3)
- net TxD: now also U4.12 (B2); no longer U4.9 (B2)
- net VIBRATION: now also U13.9 (IO0_5); no longer U13.6 (IO0_5)
- net at R7.1: now also U4.8 (OE); no longer U4.12 (OE)
- net at TP24.1, U12.3 (SDA): now also U9.13 (B1); no longer U9.10 (B1)
- net at TP25.1, U12.6 (SDC): now also U9.12 (B2); no longer U9.9 (B2)
- net at R34.1: now also U13.21 (A0); no longer U13.18 (A0)
- net at R33.1: now also U13.2 (A1); no longer U13.23 (A1)
- net at R26.1: now also U9.8 (OE); no longer U9.12 (OE)
- net OLED-MISO: no longer names the net of U2.14 (IO12)
- new net: L2.1, U11.3 (SW)
- new net: R36.2, R37.1, U11.5 (FB)
Other:
- moved on the sheet: C38, C40, TP32
